Commit message: rrbot position controller done

File: gz_rrbot_ros2/urdf/rrbot.xacro (robot description, xacro)
@@ -182,4 +182,13 @@
       <state_interface name="effort"/>
     </joint>
+    <joint name="joint2">
+      <command_interface name="position">
+        <param name="min">-6.28</param>
+        <param name="max">6.28</param>
+      </command_interface>
+      <state_interface name="position"/>
+      <state_interface name="velocity"/>
+      <state_interface name="effort"/>
+    </joint>
   </ros2_control>
   <!-- Gazebo's ros2_control plugin -->
