Commit message: custom hw done

File: gz_rrbot_ros2/urdf/rrbot_custom_hw.xacro (robot description, xacro)
@@ -56,5 +56,4 @@
     <dynamics damping="0.7"/>
   </joint>
-  <!-- Middle Link -->
   <link name="link2">
     <collision>
@@ -84,5 +83,4 @@
     <dynamics damping="0.7"/>
   </joint>
-  <!-- Top Link -->
   <link name="link3">
     <collision>
@@ -105,31 +103,4 @@
     </inertial>
   </link>
-  <!-- Hokuyo Laser
-  <joint name="hokuyo_joint" type="fixed">
-    <axis xyz="0 1 0"/>
-    <origin xyz="0 0 ${height3 - axel_offset/2}" rpy="0 0 0"/>
-    <parent link="link3"/>
-    <child link="hokuyo_link"/>
-  </joint>
-  <link name="hokuyo_link">
-    <collision>
-      <origin xyz="0 0 0" rpy="0 0 0"/>
-      <geometry>
-        <box size="0.1 0.1 0.1"/>
-      </geometry>
-    </collision>
-    <visual>
-      <origin xyz="0 0 0" rpy="0 0 0"/>
-      <geometry>
-        <mesh filename="$(find rrbot_description)/meshes/hokuyo.dae"/>
-      </geometry>
-    </visual>
-    <inertial>
-      <mass value="1e-5"/>
-      <origin xyz="0 0 0" rpy="0 0 0"/>
-      <inertia ixx="1e-6" ixy="0" ixz="0" iyy="1e-6" iyz="0" izz="1e-6"/>
-    </inertial>
-  </link>
-  -->
   <joint name="camera_joint" type="fixed">
     <axis xyz="0 1 0"/>
@@ -138,5 +109,4 @@
     <child link="camera_link"/>
   </joint>
-  <!-- Camera -->
   <link name="camera_link">
     <collision>
@@ -159,6 +129,4 @@
     </inertial>
   </link>
-  <!-- generate an optical frame http://www.ros.org/reps/rep-0103.html#suffix-frames
-   so that ros and opencv can operate on the camera frame correctly -->
   <joint name="camera_optical_joint" type="fixed">
     <!-- these values have to be these values otherwise the gazebo camera image won't
@@ -191,10 +159,3 @@
     </joint>
   </ros2_control>
-  <!-- yaml이 아닌 launch에서 param 전달 -->
-  <!-- <gazebo>
-    <plugin filename="libgazebo_ros2_control.so" name="gazebo_ros2_control">
-      <robot_sim_type>gazebo_ros2_control/GazeboSystem</robot_sim_type>
-      <parameters>$(find gz_rrbot_ros2)/config/controller_configuration.yaml</parameters>
-    </plugin>
-  </gazebo> -->
 </robot>
