Commit message: ongoing ros2_control adaptation

File: gz_rrbot_ros2/ros2_control/rrbot.ros2_control.xacro (robot description, xacro)
@@ -11,5 +11,11 @@
           <param name="max">1</param>
         </command_interface>
+        <command_interface name="velocity">
+          <param name="min">-1.0</param>
+          <param name="max">1.0</param>
+        </command_interface>
         <state_interface name="position"/>
+        <state_interface name="velocity"/>
+        <state_interface name="effort"/>
       </joint>
       <joint name="${prefix}joint2">
@@ -18,12 +24,18 @@
           <param name="max">1</param>
         </command_interface>
+        <command_interface name="velocity">
+          <param name="min">-1.0</param>
+          <param name="max">1.0</param>
+        </command_interface>
         <state_interface name="position"/>
+        <state_interface name="velocity"/>
+        <state_interface name="effort"/>
       </joint>
     </ros2_control>
-    <!-- <gazebo>
+    <gazebo>
       <plugin name="gazebo_ros2_control" filename="libgazebo_ros2_control.so">
-          <parameters>$(find dd_gazebo)/config/opensg_robot_controller.yaml</parameters>
+          <parameters>$(find gz_rrbot_ros2)/config/traj_controller.yaml</parameters>
       </plugin>
-    </gazebo> -->
+    </gazebo>
   </xacro:macro>
 </robot>

File: gz_rrbot_ros2/urdf/rrbot.materials.xacro (robot description, xacro)
@@ -4,5 +4,7 @@
 https://github.com/ros-simulation/gazebo_ros_demos/blob/kinetic-devel/rrbot_description/urdf/materials.xacro
 -->
-<robot>
+<robot xmlns:xacro="http://www.ros.org/wiki/xacro">
+  <xacro:macro name="rrbot" params="prefix *origin">
+  <xacro:property name="link_color" value="Gazebo/Silver" />
   <material name="black">
     <color rgba="0.0 0.0 0.0 1.0"/>
@@ -32,3 +34,14 @@
     <color rgba="1.0 1.0 1.0 1.0"/>
   </material>
+  <gazebo reference="${prefix}link1">
+    <material>${link_color}</material>
+    <selfCollide>false</selfCollide>
+    <!-- <gravity>true</gravity> -->
+  </gazebo>
+  <gazebo reference="${prefix}link2">
+    <material>${link_color}</material>
+    <selfCollide>false</selfCollide>
+    <!-- <gravity>true</gravity> -->
+  </gazebo>
+  </xacro:macro>
 </robot>

File: gz_rrbot_ros2/urdf/rrbot.urdf.xacro (robot description, xacro)
@@ -11,4 +11,6 @@
   <!-- Import Rviz colors -->
   <xacro:include filename="$(find gz_rrbot_ros2)/urdf/rrbot.materials.xacro" />
+  <!-- Import ros2_control -->
+  <xacro:include filename="$(find gz_rrbot_ros2)/ros2_control/rrbot.ros2_control.xacro" />
   <!-- Import RRBot ros2_control description -->
   <!-- <xacro:include filename="$(find gz_rrbot_ros2)/ros2_control/rrbot.ros2_control.xacro" /> -->
